File: 4 x MIDI Thru Box with LED.sch (EAGLE design)
At the start: 26 parts, among them IC1 7805, IC2 74AC14N, J1 xx amps, X1 MIDI, X2 MIDI, X3 MIDI, X4 MIDI, X5 MIDI

Commit message: Added BOM
Parts:
- removed D1: 1N4148, diode:DIODE-D-5
Connections:
- removed net N$6: D1.A, J1.3
- net N$8: no longer D1.C
Other:
- moved on the sheet: C1, C3, IC2P
Changed lines of the file:
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@@
 <part name="GND2" library="SparkFun" deviceset="GND" device=""/>
 <part name="LED1" library="led" deviceset="LED" device="3MM"/>
-<part name="D1" library="diode" deviceset="DIODE-" device="D-5" value="1N4148"/>
 </parts>
 <sheets>
@@
 <instance part="J1" gate="G$1" x="12.7" y="-10.16"/>
 <instance part="IC1" gate="1" x="50.8" y="-7.62"/>
-<instance part="C1" gate="G$1" x="38.1" y="-12.7"/>
-<instance part="C3" gate="G$1" x="76.2" y="-12.7"/>
-<instance part="P+2" gate="1" x="76.2" y="0"/>
+<instance part="C1" gate="G$1" x="33.02" y="-12.7"/>
+<instance part="C3" gate="G$1" x="71.12" y="-12.7"/>
+<instance part="P+2" gate="1" x="71.12" y="0"/>
 <instance part="GND3" gate="1" x="50.8" y="-25.4"/>
 <instance part="X1" gate="G$1" x="12.7" y="-53.34"/>
@@
 <instance part="P+10" gate="1" x="215.9" y="0"/>
 <instance part="GND13" gate="1" x="198.12" y="-124.46"/>
-<instance part="IC2" gate="P" x="99.06" y="-10.16"/>
-<instance part="P+1" gate="1" x="99.06" y="0"/>
-<instance part="GND1" gate="1" x="99.06" y="-20.32"/>
+<instance part="IC2" gate="P" x="93.98" y="-10.16"/>
+<instance part="P+1" gate="1" x="93.98" y="0"/>
+<instance part="GND1" gate="1" x="93.98" y="-20.32"/>
 <instance part="C2" gate="G$1" x="71.12" y="-38.1" rot="R270"/>
 <instance part="GND2" gate="1" x="60.96" y="-43.18"/>
 <instance part="LED1" gate="G$1" x="180.34" y="-10.16" rot="R270"/>
-<instance part="D1" gate="G$1" x="25.4" y="-7.62"/>
 </instances>
 <busses>
@@
 <net name="GND" class="0">
 <segment>
-<wire x1="38.1" y1="-17.78" x2="38.1" y2="-20.32" width="0.1524" layer="91"/>
-<wire x1="50.8" y1="-20.32" x2="76.2" y2="-20.32" width="0.1524" layer="91"/>
-<wire x1="76.2" y1="-20.32" x2="76.2" y2="-17.78" width="0.1524" layer="91"/>
+<wire x1="33.02" y1="-17.78" x2="33.02" y2="-20.32" width="0.1524" layer="91"/>
+<wire x1="50.8" y1="-20.32" x2="71.12" y2="-20.32" width="0.1524" layer="91"/>
+<wire x1="71.12" y1="-20.32" x2="71.12" y2="-17.78" width="0.1524" layer="91"/>
 <wire x1="50.8" y1="-15.24" x2="50.8" y2="-20.32" width="0.1524" layer="91"/>
 <wire x1="50.8" y1="-20.32" x2="50.8" y2="-22.86" width="0.1524" layer="91"/>
@@
 <pinref part="J1" gate="G$1" pin="1"/>
 <wire x1="17.78" y1="-12.7" x2="17.78" y2="-20.32" width="0.1524" layer="91"/>
-<wire x1="17.78" y1="-20.32" x2="38.1" y2="-20.32" width="0.1524" layer="91"/>
-<wire x1="38.1" y1="-20.32" x2="50.8" y2="-20.32" width="0.1524" layer="91"/>
-<junction x="38.1" y="-20.32"/>
+<wire x1="17.78" y1="-20.32" x2="33.02" y2="-20.32" width="0.1524" layer="91"/>
+<wire x1="33.02" y1="-20.32" x2="50.8" y2="-20.32" width="0.1524" layer="91"/>
+<junction x="33.02" y="-20.32"/>
 </segment>
 <segment>
@@
 <net name="N$8" class="0">
 <segment>
-<wire x1="38.1" y1="-10.16" x2="38.1" y2="-7.62" width="0.1524" layer="91"/>
-<wire x1="38.1" y1="-7.62" x2="43.18" y2="-7.62" width="0.1524" layer="91"/>
+<wire x1="33.02" y1="-10.16" x2="33.02" y2="-7.62" width="0.1524" layer="91"/>
+<wire x1="33.02" y1="-7.62" x2="43.18" y2="-7.62" width="0.1524" layer="91"/>
 <pinref part="C1" gate="G$1" pin="+"/>
 <pinref part="IC1" gate="1" pin="IN"/>
-<pinref part="D1" gate="G$1" pin="C"/>
-<wire x1="27.94" y1="-7.62" x2="38.1" y2="-7.62" width="0.1524" layer="91"/>
-<junction x="38.1" y="-7.62"/>
+<wire x1="17.78" y1="-7.62" x2="33.02" y2="-7.62" width="0.1524" layer="91"/>
+<junction x="33.02" y="-7.62"/>
 </segment>
 </net>
 <net name="+5V" class="0">
 <segment>
-<wire x1="76.2" y1="-7.62" x2="76.2" y2="-2.54" width="0.1524" layer="91"/>
-<wire x1="76.2" y1="-10.16" x2="76.2" y2="-7.62" width="0.1524" layer="91"/>
-<wire x1="76.2" y1="-7.62" x2="58.42" y2="-7.62" width="0.1524" layer="91"/>
-<junction x="76.2" y="-7.62"/>
+<wire x1="71.12" y1="-7.62" x2="71.12" y2="-2.54" width="0.1524" layer="91"/>
+<wire x1="71.12" y1="-10.16" x2="71.12" y2="-7.62" width="0.1524" layer="91"/>
+<wire x1="71.12" y1="-7.62" x2="58.42" y2="-7.62" width="0.1524" layer="91"/>
+<junction x="71.12" y="-7.62"/>
 <pinref part="P+2" gate="1" pin="+5V"/>
 <pinref part="C3" gate="G$1" pin="+"/>
@@
 </segment>
 </net>
-<net name="N$6" class="0">
-<segment>
-<pinref part="J1" gate="G$1" pin="3"/>
-<pinref part="D1" gate="G$1" pin="A"/>
-<wire x1="17.78" y1="-7.62" x2="22.86" y2="-7.62" width="0.1524" layer="91"/>
-</segment>
-</net>

Commit message: Started PCB design
Parts:
- C1: device rcl:CPOL-USE7.5-16 -> rcl:CPOL-EUTT2D6
- C2: device rcl:CPOL-USE7.5-16 -> rcl:C-EU025-024X044
- C3: device rcl:CPOL-USE2.5-7 -> rcl:CPOL-EUTT2D6
Connections:
- net +5V: now also C2.1; no longer C2.+
- net GND: now also C2.2; no longer C2.-
Changed lines of the file:
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@@
 <part name="J1" library="con-jack2" deviceset="JACK-PLUG" device="2" value="xx amps"/>
 <part name="IC1" library="v-reg" deviceset="78XXS" device="" value="7805"/>
-<part name="C1" library="rcl" deviceset="CPOL-US" device="E7.5-16" value="47uF"/>
-<part name="C3" library="rcl" deviceset="CPOL-US" device="E2.5-7" value="0.1uF"/>
+<part name="C1" library="rcl" deviceset="CPOL-EU" device="TT2D6" value="47uF"/>
+<part name="C3" library="rcl" deviceset="CPOL-EU" device="TT2D6" value="0.1uF"/>
 <part name="P+2" library="supply1" deviceset="+5V" device=""/>
 <part name="GND3" library="SparkFun" deviceset="GND" device=""/>
@@
 <part name="P+1" library="supply1" deviceset="+5V" device=""/>
 <part name="GND1" library="SparkFun" deviceset="GND" device=""/>
-<part name="C2" library="rcl" deviceset="CPOL-US" device="E7.5-16" value="100nF"/>
+<part name="C2" library="rcl" deviceset="C-EU" device="025-024X044" value="100nF"/>
 <part name="GND2" library="SparkFun" deviceset="GND" device=""/>
 <part name="LED1" library="led" deviceset="LED" device="3MM"/>
@@
 </segment>
 <segment>
-<pinref part="C2" gate="G$1" pin="-"/>
+<pinref part="C2" gate="G$1" pin="2"/>
 <pinref part="GND2" gate="1" pin="GND"/>
 <wire x1="66.04" y1="-38.1" x2="60.96" y2="-38.1" width="0.1524" layer="91"/>
@@
 <pinref part="C1" gate="G$1" pin="+"/>
 <pinref part="IC1" gate="1" pin="IN"/>
-<wire x1="17.78" y1="-7.62" x2="33.02" y2="-7.62" width="0.1524" layer="91"/>
+<wire x1="12.7" y1="-7.62" x2="33.02" y2="-7.62" width="0.1524" layer="91"/>
 <junction x="33.02" y="-7.62"/>
 </segment>
@@
 <wire x1="78.74" y1="-38.1" x2="73.66" y2="-38.1" width="0.1524" layer="91"/>
 <junction x="78.74" y="-38.1"/>
-<pinref part="C2" gate="G$1" pin="+"/>
+<pinref part="C2" gate="G$1" pin="1"/>
 </segment>
 </net>

Commit message: Completed PCB design
Parts:
- added LED2: Red, led:LED3MM
- added R12: 220, rcl:R-US_0204/7
- C2: value 100nF -> 0.1uF; device rcl:C-EU025-024X044 -> rcl:CPOL-EUTT2D6
- C3: value 0.1uF -> 100nF; device rcl:CPOL-EUTT2D6 -> rcl:C-EU025-024X044
- LED1: value (none) -> Green
- R2: value 820 -> 330
- R3: value 330 -> 820
- R4: value 220 -> 330
- renumbered D2 to D1
Connections:
- removed net N$8: C1.+, IC1.IN
- new net N$6: C1.+, IC1.IN, J1.3
- new net N$9: LED1.C, R2.1
- net +5V: now also C2.+, C3.1, LED2.A, R12.1, R3.2; no longer C2.1, C3.+, R2.2, R8.1
- net GND: now also C2.-, C3.2, R2.2; no longer C2.2, C3.-
- net MIDI_IN: now also R3.1; no longer R2.1
- net N$1: now also R5.2; no longer R4.2
- net N$2: now also R7.2; no longer R6.2
- net N$21: now also R7.1; no longer R6.1
- net N$22: now also R6.2; no longer R5.2
- net N$23: now also R5.1; no longer R4.1
- net N$26: now also R8.2; no longer R7.2
- net N$3: now also R8.1; no longer R7.1
- net N$4: now also R9.2; no longer R8.2
- net N$41: now also R6.1; no longer R5.1
- net N$5: now also LED2.C, R4.1; no longer LED1.C, R3.1
- net N$52: now also R12.2; no longer R11.2
- net N$53: now also R11.2; no longer R10.2
- net N$54: now also R10.2; no longer R9.2
- net N$65: now also R4.2; no longer R3.2
Other:
- moved on the sheet: C1, IC1, IC2P, J1, LED1, R10, R11, R2, R3, R4, R5, R6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

Commit message: Version 1.0
Parts:
- J1: value xx amps -> 9V DC
- LED1: value Green -> Power
- LED2: value Red -> Midi In
Changed lines of the file:
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@@
 </classes>
 <parts>
-<part name="J1" library="con-jack2" deviceset="JACK-PLUG" device="2" value="xx amps"/>
+<part name="J1" library="con-jack2" deviceset="JACK-PLUG" device="2" value="9V DC"/>
 <part name="IC1" library="v-reg" deviceset="78XXS" device="" value="7805"/>
 <part name="C1" library="rcl" deviceset="CPOL-EU" device="TT2D6" value="47uF"/>
@@
 <part name="C3" library="rcl" deviceset="C-EU" device="025-024X044" value="100nF"/>
 <part name="GND2" library="SparkFun" deviceset="GND" device=""/>
-<part name="LED2" library="led" deviceset="LED" device="3MM" value="Red"/>
-<part name="LED1" library="led" deviceset="LED" device="3MM" value="Green"/>
+<part name="LED2" library="led" deviceset="LED" device="3MM" value="Midi In"/>
+<part name="LED1" library="led" deviceset="LED" device="3MM" value="Power"/>
 <part name="R2" library="rcl" deviceset="R-US_" device="0204/7" value="330"/>
 </parts>
